File: hardware/pcbs/atmega2560-basebord/atmega2560-basebord.sch (KiCad schematic (older format))
At the start: 0 parts

Commit message: Add decoupling capacitors
Parts:
- added C? (x3): 0.1uF, symbol C
- added U?: ATMEGA2560-16AU, TQFP100, symbol ATMEGA2560-16AU
Connections:
- net labels added: +5V, GND
- wire segments 0 -> 22
Changed lines of the file:
@@
 LIBS:contrib
 LIBS:valves
+LIBS:atmega2560-basebord-cache
 EELAYER 25 0
 EELAYER END
@@
 Comment4 ""
 $EndDescr
+$Comp
+L ATMEGA2560-16AU U?
+U 1 1 5B4B7E8F
+P 2300 3900
+F 0 "U?" H 1150 6700 50  0000 L BNN
+F 1 "ATMEGA2560-16AU" H 3000 1050 50  0000 L BNN
+F 2 "TQFP100" H 2300 3900 50  0001 C CIN
+F 3 "" H 2300 3900 50  0001 C CNN
+	1    2300 3900
+	1    0    0    -1
+$EndComp
+$Comp
+L +5V #PWR?
+U 1 1 5B4B88FD
+P 1650 900
+F 0 "#PWR?" H 1650 750 50  0001 C CNN
+F 1 "+5V" H 1650 1040 50  0000 C CNN
+F 2 "" H 1650 900 50  0001 C CNN
+F 3 "" H 1650 900 50  0001 C CNN
+	1    1650 900
+	1    0    0    -1
+$EndComp
+$Comp
+L GND #PWR?
+U 1 1 5B4B89DB
+P 1900 6950
+F 0 "#PWR?" H 1900 6700 50  0001 C CNN
+F 1 "GND" H 1900 6800 50  0000 C CNN
+F 2 "" H 1900 6950 50  0001 C CNN
+F 3 "" H 1900 6950 50  0001 C CNN
+	1    1900 6950
+	1    0    0    -1
+$EndComp
+Wire Wire Line
+	1650 900  1650 950
+Wire Wire Line
+	1650 950  2450 950
+Wire Wire Line
+	1950 950  1950 1000
+Wire Wire Line
+	2050 950  2050 1000
+Connection ~ 1950 950
+Wire Wire Line
+	2150 950  2150 1000
+Connection ~ 2050 950
+Wire Wire Line
+	2250 950  2250 1000
+Connection ~ 2150 950
+Wire Wire Line
+	2450 950  2450 1000
+Connection ~ 2250 950
+Wire Wire Line
+	1900 6950 1900 6850
+Wire Wire Line
+	1900 6850 2550 6850
+Wire Wire Line
+	2150 6850 2150 6800
+Wire Wire Line
+	2250 6850 2250 6800
+Connection ~ 2150 6850
+Wire Wire Line
+	2350 6850 2350 6800
+Connection ~ 2250 6850
+Wire Wire Line
+	2450 6850 2450 6800
+Connection ~ 2350 6850
+Wire Wire Line
+	2550 6850 2550 6800
+Connection ~ 2450 6850
+$Comp
+L C C?
+U 1 1 5B4B95A0
+P 4850 1650
+F 0 "C?" H 4875 1750 50  0000 L CNN
+F 1 "0.1uF" H 4875 1550 50  0000 L CNN
+F 2 "" H 4888 1500 50  0001 C CNN
+F 3 "" H 4850 1650 50  0001 C CNN
+	1    4850 1650
+	1    0    0    -1
+$EndComp
+$Comp
+L C C?
+U 1 1 5B4B961F
+P 5350 1650
+F 0 "C?" H 5375 1750 50  0000 L CNN
+F 1 "0.1uF" H 5375 1550 50  0000 L CNN
+F 2 "" H 5388 1500 50  0001 C CNN
+F 3 "" H 5350 1650 50  0001 C CNN
+	1    5350 1650
+	1    0    0    -1
+$EndComp
+$Comp
+L C C?
+U 1 1 5B4B9643
+P 5800 1650
+F 0 "C?" H 5825 1750 50  0000 L CNN
+F 1 "0.1uF" H 5825 1550 50  0000 L CNN
+F 2 "" H 5838 1500 50  0001 C CNN
+F 3 "" H 5800 1650 50  0001 C CNN
+	1    5800 1650
+	1    0    0    -1
+$EndComp
+Wire Wire Line
+	4850 1500 4850 1350
+Wire Wire Line
+	4850 1350 5800 1350
+Wire Wire Line
+	5350 1150 5350 1500
+Wire Wire Line
+	5800 1350 5800 1500
+Connection ~ 5350 1350
+Wire Wire Line
+	5800 1950 5800 1800
+Wire Wire Line
+	4850 1950 5800 1950
+Wire Wire Line
+	5350 1800 5350 2100
+Wire Wire Line
+	4850 1950 4850 1800
+Connection ~ 5350 1950
+$Comp
+L GND #PWR?
+U 1 1 5B4B9704
+P 5350 2100
+F 0 "#PWR?" H 5350 1850 50  0001 C CNN
+F 1 "GND" H 5350 1950 50  0000 C CNN
+F 2 "" H 5350 2100 50  0001 C CNN
+F 3 "" H 5350 2100 50  0001 C CNN
+	1    5350 2100
+	1    0    0    -1
+$EndComp
+$Comp
+L +5V #PWR?
+U 1 1 5B4B974E
+P 5350 1150
+F 0 "#PWR?" H 5350 1000 50  0001 C CNN
+F 1 "+5V" H 5350 1290 50  0000 C CNN
+F 2 "" H 5350 1150 50  0001 C CNN
+F 3 "" H 5350 1150 50  0001 C CNN
+	1    5350 1150
+	1    0    0    -1
+$EndComp
 $EndSCHEMATC

Commit message: Resize schematics and add reset line
Parts:
- added C?: 0.1uF, symbol C
- added R?: 10K, symbol R
Connections:
- net labels added: RST
- wire segments 22 -> 28
Changed lines of the file:
@@
 EELAYER 25 0
 EELAYER END
-$Descr A4 11693 8268
+$Descr User 8819 8268
 encoding utf-8
 Sheet 1 1
@@
 L ATMEGA2560-16AU U?
 U 1 1 5B4B7E8F
-P 2300 3900
-F 0 "U?" H 1150 6700 50  0000 L BNN
-F 1 "ATMEGA2560-16AU" H 3000 1050 50  0000 L BNN
-F 2 "TQFP100" H 2300 3900 50  0001 C CIN
-F 3 "" H 2300 3900 50  0001 C CNN
-	1    2300 3900
+P 2500 4150
+F 0 "U?" H 1350 6950 50  0000 L BNN
+F 1 "ATMEGA2560-16AU" H 3200 1300 50  0000 L BNN
+F 2 "TQFP100" H 2500 4150 50  0001 C CIN
+F 3 "" H 2500 4150 50  0001 C CNN
+	1    2500 4150
 	1    0    0    -1
 $EndComp
@@
 L +5V #PWR?
 U 1 1 5B4B88FD
-P 1650 900
-F 0 "#PWR?" H 1650 750 50  0001 C CNN
-F 1 "+5V" H 1650 1040 50  0000 C CNN
-F 2 "" H 1650 900 50  0001 C CNN
-F 3 "" H 1650 900 50  0001 C CNN
-	1    1650 900
+P 1850 1150
+F 0 "#PWR?" H 1850 1000 50  0001 C CNN
+F 1 "+5V" H 1850 1290 50  0000 C CNN
+F 2 "" H 1850 1150 50  0001 C CNN
+F 3 "" H 1850 1150 50  0001 C CNN
+	1    1850 1150
 	1    0    0    -1
 $EndComp
@@
 L GND #PWR?
 U 1 1 5B4B89DB
-P 1900 6950
-F 0 "#PWR?" H 1900 6700 50  0001 C CNN
-F 1 "GND" H 1900 6800 50  0000 C CNN
-F 2 "" H 1900 6950 50  0001 C CNN
-F 3 "" H 1900 6950 50  0001 C CNN
-	1    1900 6950
-	1    0    0    -1
-$EndComp
-Wire Wire Line
-	1650 900  1650 950
-Wire Wire Line
-	1650 950  2450 950
-Wire Wire Line
-	1950 950  1950 1000
-Wire Wire Line
-	2050 950  2050 1000
-Connection ~ 1950 950
-Wire Wire Line
-	2150 950  2150 1000
-Connection ~ 2050 950
-Wire Wire Line
-	2250 950  2250 1000
-Connection ~ 2150 950
-Wire Wire Line
-	2450 950  2450 1000
-Connection ~ 2250 950
-Wire Wire Line
-	1900 6950 1900 6850
-Wire Wire Line
-	1900 6850 2550 6850
-Wire Wire Line
-	2150 6850 2150 6800
-Wire Wire Line
-	2250 6850 2250 6800
-Connection ~ 2150 6850
-Wire Wire Line
-	2350 6850 2350 6800
-Connection ~ 2250 6850
-Wire Wire Line
-	2450 6850 2450 6800
-Connection ~ 2350 6850
-Wire Wire Line
-	2550 6850 2550 6800
-Connection ~ 2450 6850
+P 2100 7200
+F 0 "#PWR?" H 2100 6950 50  0001 C CNN
+F 1 "GND" H 2100 7050 50  0000 C CNN
+F 2 "" H 2100 7200 50  0001 C CNN
+F 3 "" H 2100 7200 50  0001 C CNN
+	1    2100 7200
+	1    0    0    -1
+$EndComp
 $Comp
 L C C?
 U 1 1 5B4B95A0
-P 4850 1650
-F 0 "C?" H 4875 1750 50  0000 L CNN
-F 1 "0.1uF" H 4875 1550 50  0000 L CNN
-F 2 "" H 4888 1500 50  0001 C CNN
-F 3 "" H 4850 1650 50  0001 C CNN
-	1    4850 1650
+P 5550 1500
+F 0 "C?" H 5575 1600 50  0000 L CNN
+F 1 "0.1uF" H 5575 1400 50  0000 L CNN
+F 2 "" H 5588 1350 50  0001 C CNN
+F 3 "" H 5550 1500 50  0001 C CNN
+	1    5550 1500
 	1    0    0    -1
 $EndComp
@@
 L C C?
 U 1 1 5B4B961F
-P 5350 1650
-F 0 "C?" H 5375 1750 50  0000 L CNN
-F 1 "0.1uF" H 5375 1550 50  0000 L CNN
-F 2 "" H 5388 1500 50  0001 C CNN
-F 3 "" H 5350 1650 50  0001 C CNN
-	1    5350 1650
+P 6050 1500
+F 0 "C?" H 6075 1600 50  0000 L CNN
+F 1 "0.1uF" H 6075 1400 50  0000 L CNN
+F 2 "" H 6088 1350 50  0001 C CNN
+F 3 "" H 6050 1500 50  0001 C CNN
+	1    6050 1500
 	1    0    0    -1
 $EndComp
@@
 L C C?
 U 1 1 5B4B9643
-P 5800 1650
-F 0 "C?" H 5825 1750 50  0000 L CNN
-F 1 "0.1uF" H 5825 1550 50  0000 L CNN
-F 2 "" H 5838 1500 50  0001 C CNN
-F 3 "" H 5800 1650 50  0001 C CNN
-	1    5800 1650
-	1    0    0    -1
-$EndComp
-Wire Wire Line
-	4850 1500 4850 1350
-Wire Wire Line
-	4850 1350 5800 1350
-Wire Wire Line
-	5350 1150 5350 1500
-Wire Wire Line
-	5800 1350 5800 1500
-Connection ~ 5350 1350
-Wire Wire Line
-	5800 1950 5800 1800
-Wire Wire Line
-	4850 1950 5800 1950
-Wire Wire Line
-	5350 1800 5350 2100
-Wire Wire Line
-	4850 1950 4850 1800
-Connection ~ 5350 1950
+P 6500 1500
+F 0 "C?" H 6525 1600 50  0000 L CNN
+F 1 "0.1uF" H 6525 1400 50  0000 L CNN
+F 2 "" H 6538 1350 50  0001 C CNN
+F 3 "" H 6500 1500 50  0001 C CNN
+	1    6500 1500
+	1    0    0    -1
+$EndComp
 $Comp
 L GND #PWR?
 U 1 1 5B4B9704
-P 5350 2100
-F 0 "#PWR?" H 5350 1850 50  0001 C CNN
-F 1 "GND" H 5350 1950 50  0000 C CNN
-F 2 "" H 5350 2100 50  0001 C CNN
-F 3 "" H 5350 2100 50  0001 C CNN
-	1    5350 2100
+P 6050 1950
+F 0 "#PWR?" H 6050 1700 50  0001 C CNN
+F 1 "GND" H 6050 1800 50  0000 C CNN
+F 2 "" H 6050 1950 50  0001 C CNN
+F 3 "" H 6050 1950 50  0001 C CNN
+	1    6050 1950
 	1    0    0    -1
 $EndComp
@@
 L +5V #PWR?
 U 1 1 5B4B974E
-P 5350 1150
-F 0 "#PWR?" H 5350 1000 50  0001 C CNN
-F 1 "+5V" H 5350 1290 50  0000 C CNN
-F 2 "" H 5350 1150 50  0001 C CNN
-F 3 "" H 5350 1150 50  0001 C CNN
-	1    5350 1150
-	1    0    0    -1
-$EndComp
+P 6050 1000
+F 0 "#PWR?" H 6050 850 50  0001 C CNN
+F 1 "+5V" H 6050 1140 50  0000 C CNN
+F 2 "" H 6050 1000 50  0001 C CNN
+F 3 "" H 6050 1000 50  0001 C CNN
+	1    6050 1000
+	1    0    0    -1
+$EndComp
+$Comp
+L R R?
+U 1 1 5B4B9879
+P 5700 3050
+F 0 "R?" V 5780 3050 50  0000 C CNN
+F 1 "10K" V 5700 3050 50  0000 C CNN
+F 2 "" V 5630 3050 50  0001 C CNN
+F 3 "" H 5700 3050 50  0001 C CNN
+	1    5700 3050
+	0    1    1    0
+$EndComp
+$Comp
+L +5V #PWR?
+U 1 1 5B4B9915
+P 5100 3200
+F 0 "#PWR?" H 5100 3050 50  0001 C CNN
+F 1 "+5V" H 5100 3340 50  0000 C CNN
+F 2 "" H 5100 3200 50  0001 C CNN
+F 3 "" H 5100 3200 50  0001 C CNN
+	1    5100 3200
+	1    0    0    -1
+$EndComp
+$Comp
+L C C?
+U 1 1 5B4B996D
+P 6050 3400
+F 0 "C?" H 6075 3500 50  0000 L CNN
+F 1 "0.1uF" H 6075 3300 50  0000 L CNN
+F 2 "" H 6088 3250 50  0001 C CNN
+F 3 "" H 6050 3400 50  0001 C CNN
+	1    6050 3400
+	1    0    0    -1
+$EndComp
+$Comp
+L GND #PWR?
+U 1 1 5B4B99D9
+P 6050 3800
+F 0 "#PWR?" H 6050 3550 50  0001 C CNN
+F 1 "GND" H 6050 3650 50  0000 C CNN
+F 2 "" H 6050 3800 50  0001 C CNN
+F 3 "" H 6050 3800 50  0001 C CNN
+	1    6050 3800
+	1    0    0    -1
+$EndComp
+Text GLabel 6450 3050 2    60   Input ~ 0
+RST
+Wire Wire Line
+	1850 1150 1850 1200
+Wire Wire Line
+	1850 1200 2650 1200
+Wire Wire Line
+	2150 1200 2150 1250
+Wire Wire Line
+	2250 1200 2250 1250
+Connection ~ 2150 1200
+Wire Wire Line
+	2350 1200 2350 1250
+Connection ~ 2250 1200
+Wire Wire Line
+	2450 1200 2450 1250
+Connection ~ 2350 1200
+Wire Wire Line
+	2650 1200 2650 1250
+Connection ~ 2450 1200
+Wire Wire Line
+	2100 7200 2100 7100
+Wire Wire Line
+	2100 7100 2750 7100
+Wire Wire Line
+	2350 7100 2350 7050
+Wire Wire Line
+	2450 7100 2450 7050
+Connection ~ 2350 7100
+Wire Wire Line
+	2550 7100 2550 7050
+Connection ~ 2450 7100
+Wire Wire Line
+	2650 7100 2650 7050
+Connection ~ 2550 7100
+Wire Wire Line
+	2750 7100 2750 7050
+Connection ~ 2650 7100
+Wire Wire Line
+	5550 1350 5550 1200
+Wire Wire Line
+	5550 1200 6500 1200
+Wire Wire Line
+	6050 1000 6050 1350
+Wire Wire Line
+	6500 1200 6500 1350
+Connection ~ 6050 1200
+Wire Wire Line
+	6500 1800 6500 1650
+Wire Wire Line
+	5550 1800 6500 1800
+Wire Wire Line
+	6050 1650 6050 1950
+Wire Wire Line
+	5550 1800 5550 1650
+Connection ~ 6050 1800
+Wire Wire Line
+	5250 2950 5250 3050
+Wire Wire Line
+	5250 3050 5550 3050
+Wire Wire Line
+	5850 3050 6450 3050
+Wire Wire Line
+	6050 3050 6050 3250
+Wire Wire Line
+	6050 3800 6050 3550
+Connection ~ 6050 3050
+Text GLabel 1100 1550 0    60   Input ~ 0
+RST
+Wire Wire Line
+	1100 1550 1200 1550
+Wire Notes Line
+	4100 6500 4100 550
 $EndSCHEMATC
