File: hardware/-pcbs/lpkf-test/lpkf-test.kicad_pcb (KiCad board)
At the start: 2 copper layers, 0 parts

Commit message: Route pcb
Parts:
- added C1: 0.1uF, Capacitors_SMD:C_0603_HandSoldering, F.Cu at (62.7, 82.7)
- added C2: 0.1uF, Capacitors_SMD:C_0603_HandSoldering, F.Cu at (72.3, 82.7)
- added C3: 0.1uF, Capacitors_SMD:C_0603_HandSoldering, F.Cu at (67.4, 82.7)
- added J1: 02x04, Pin_Headers:Pin_Header_Straight_2x04_Pitch2.54mm, F.Cu at (61.2, 63.0)
- added R1: 10K, Resistors_SMD:R_0603_HandSoldering, F.Cu at (80.9, 79.5)
- added R2: 10K, Resistors_SMD:R_0603_HandSoldering, F.Cu at (66.5, 76.4)
- added U1: ATMEGA168PA-AU, Housings_QFP:TQFP-32_7x7mm_Pitch0.8mm, F.Cu at (76.9, 67.1)
Routing:
- net GND: track 0.00 -> 82.7 mm, vias 0 -> 4
- net +5V: track 0.00 -> 76.9 mm, vias 0 -> 4
- net Net-(J1-Pad3): track 0.00 -> 62.3 mm, vias 0 -> 2
- net /SDA: track 0.00 -> 58.8 mm, vias 0 -> 3
- net Net-(J1-Pad4): track 0.00 -> 49.8 mm, vias 0 -> 5
- net /SCL: track 0.00 -> 43.1 mm
- net Net-(J1-Pad2): track 0.00 -> 22.6 mm, vias 0 -> 2
- net Net-(J1-Pad1): track 0.00 -> 20.0 mm, vias 0 -> 2
Other:
- board outline added: 30.5 x 30.5 mm
- board text added: "araTest"
