File: hardware/ecg-baseboard/ecg-baseboard.kicad_pcb (KiCad board)
At the start: 2 copper layers, 40 x 100 mm, 9 parts, among them J1 Screw_Terminal_01x04, J2 Protocentral MAX30003, J3 Conn_01x06

Commit message: [hw] Update footprint of ECG Baseboard project
Parts:
- G***: footprint ecg-baseboard:heart-logo -> ECG-BASEBOARD:heart-logo
